Commit message: finish diff_drive_car in gazebo

File: robot_gazebo/urdf/my_laser.urdf.xacro (robot description, xacro)
@@ -1,5 +1,5 @@
 <!-- 雷达 -->
 <robot name="my_laser" xmlns:xacro="http://wiki.ros.org/xacro">
-    <xacro:property name="support_length" value="0.15" /> <!-- 支架长度 -->
+    <xacro:property name="support_length" value="0.05" /> <!-- 支架长度 -->
     <xacro:property name="support_radius" value="0.01" /> <!-- 支架半径 -->
     <xacro:property name="support_x" value="0.0" /> <!-- 支架安装的x坐标 -->
