Commit message: complete gazebo vitrual monitor

File: robot_gazebo/urdf/move.urdf.xacro (robot description, xacro)
@@ -1,24 +1,54 @@
 <robot name="my_car_move" xmlns:xacro="http://www.ros.org/wiki/xacro">
-  <!-- 接口声明 -->
+  <!-- ========== 引用 my_base 的底盘和轮子属性 ========== -->
+  <xacro:include filename="my_base.urdf.xacro"/>
+  <xacro:my_base />
+  <!-- ========== ros2_control 定义 ========== -->
   <ros2_control name="GazeboSystem" type="system">
     <hardware>
-        <plugin>gazebo_ros2_control/GazeboSystem</plugin>
+      <plugin>gazebo_ros2_control/GazeboSystem</plugin>
     </hardware>
-    <joint name="left_wheel2base_link">
+    <!-- 四个麦轮 joint -->
+    <joint name="front_left_wheel_joint">
       <command_interface name="velocity"/>
-      <state_interface name="position"/>
       <state_interface name="velocity"/>
     </joint>
-    <joint name="right_wheel2base_link">
+    <joint name="front_right_wheel_joint">
       <command_interface name="velocity"/>
-      <state_interface name="position"/>
+      <state_interface name="velocity"/>
+    </joint>
+    <joint name="rear_left_wheel_joint">
+      <command_interface name="velocity"/>
+      <state_interface name="velocity"/>
+    </joint>
+    <joint name="rear_right_wheel_joint">
+      <command_interface name="velocity"/>
       <state_interface name="velocity"/>
     </joint>
   </ros2_control>
-  <!-- ros2_control 插件加载 -->
   <gazebo>
-  <plugin name="gazebo_ros2_control" filename="libgazebo_ros2_control.so">
-    <parameters>$(find robot_gazebo)/config/ros2_config.yaml</parameters>
-  </plugin>
-</gazebo>
+    <plugin name="gazebo_ros2_control" filename="libgazebo_ros2_control.so">
+      <parameters>/home/hiro/ros2/AIC_car_2025/robot_gazebo/urdf/mecanum_controllers.yaml</parameters>
+    </plugin>
+  </gazebo>
+  <controller name="mecanum_controller" type="mecanum_drive_controller/MecanumDriveController">
+    <ros>
+      <namespace>/</namespace>
+      <!-- <parameters>
+        <param name="front_left_wheel_command_joint_name" value="front_left_wheel_joint"/>
+        <param name="front_right_wheel_command_joint_name" value="front_right_wheel_joint"/>
+        <param name="rear_left_wheel_command_joint_name" value="rear_left_wheel_joint"/>
+        <param name="rear_right_wheel_command_joint_name" value="rear_right_wheel_joint"/>
+        <param name="front_left_wheel_state_joint_name" value="front_left_wheel_joint"/>
+        <param name="front_right_wheel_state_joint_name" value="front_right_wheel_joint"/>
+        <param name="rear_left_wheel_state_joint_name" value="rear_left_wheel_joint"/>
+        <param name="rear_right_wheel_state_joint_name" value="rear_right_wheel_joint"/>
+        <param name="wheel_radius" value="0.05"/>
+        <param name="wheel_separation_x" value="0.3"/>
+        <param name="wheel_separation_y" value="0.25"/>
+        <param name="command_interface" value="['velocity']"/>
+        <param name="state_interface" value="['velocity']"/>
+        <param name="publish_rate" value="50.0"/>
+      </parameters> -->
+    </ros>
+  </controller>
 </robot>

File: robot_gazebo/urdf/my_base.urdf.xacro (robot description, xacro)
@@ -1,30 +1,12 @@
-<!--
-    使用 xacro 优化 URDF 版的小车底盘实现：
-    1.将一些常量、变量封装为 xacro:property PI 值、小车底盘半径、离地间距、车轮半径、宽度
-    2.使用宏封装驱动轮以及支撑轮实现，调用生成驱动轮与支撑轮
--->
-<!-- 根标签，必须声明 xmlns:xacro -->
 <robot name="my_base" xmlns:xacro="http://www.ros.org/wiki/xacro">
-    <!-- 封装变量、常量 -->
-    <!-- PI 值设置精度需要高一些，否则后续车轮翻转量计算时，可能会出现肉眼不能察觉的车轮倾斜，从而导致模型抖动 -->
-    <xacro:property name="PI" value="3.1415926"/>
-    <!-- 宏:黑色设置 -->
+  <xacro:macro name="my_base">
+    <!-- 宏:颜色设置 -->
     <material name="black">
         <color rgba="0.0 0.0 0.0 1.0" />
     </material>
-    <!-- 底盘属性 -->
-    <xacro:property name="base_footprint_radius" value="0.001" /> <!-- base_footprint 半径  -->
-    <xacro:property name="base_link_radius" value="0.1" /> <!-- base_link 半径 -->
-    <xacro:property name="base_link_length" value="0.08" /> <!-- base_link 长 -->
-    <xacro:property name="earth_space" value="0.015" /> <!-- 离地间距 -->
-    <xacro:property name="base_link_m" value="0.5" /> <!-- 质量  -->
-    <!-- 底盘 -->
-    <link name="base_footprint">
-      <visual>
-        <geometry>
-          <sphere radius="${base_footprint_radius}" />
-        </geometry>
-      </visual>
-    </link>
+    <material name="yellow">
+        <color rgba="1.0 1.0 0.0 1.0" />
+    </material>
+    <!-- 底盘主体 -->
     <link name="base_link">
       <visual>
@@ -37,27 +19,7 @@
         </material>
       </visual>
-      <collision>
-        <geometry>
-          <cylinder radius="${base_link_radius}" length="${base_link_length}" />
-        </geometry>
-        <origin xyz="0 0 0" rpy="0 0 0" />
-      </collision>
-      <xacro:cylinder_inertial_matrix m="${base_link_m}" r="${base_link_radius}" h="${base_link_length}" />
     </link>
-    <joint name="base_link2base_footprint" type="fixed">
-      <parent link="base_footprint" />
-      <child link="base_link" />
-      <origin xyz="0 0 ${earth_space + base_link_length / 2 }" />
-    </joint>
-    <gazebo reference="base_link">
-        <material>Gazebo/Yellow</material>
-    </gazebo>
-    <!-- 驱动轮 -->
-    <!-- 驱动轮属性 -->
-    <xacro:property name="wheel_radius" value="0.0325" /><!-- 半径 -->
-    <xacro:property name="wheel_length" value="0.015" /><!-- 宽度 -->
-    <xacro:property name="wheel_m" value="0.05" /> <!-- 质量  -->
-    <!-- 驱动轮宏实现 -->
-    <xacro:macro name="add_wheels" params="name flag">
+    <!-- 四个驱动轮宏 -->
+    <xacro:macro name="add_wheel" params="name x y">
       <link name="${name}_wheel">
         <visual>
@@ -65,6 +27,6 @@
             <cylinder radius="${wheel_radius}" length="${wheel_length}" />
           </geometry>
-          <origin xyz="0.0 0.0 0.0" rpy="${PI / 2} 0.0 0.0" />
-          <material name="black" />
+          <origin xyz="0 0 0" rpy="${PI/2} 0 0" />
+          <material name="yellow"/>
         </visual>
         <collision>
@@ -72,53 +34,23 @@
             <cylinder radius="${wheel_radius}" length="${wheel_length}" />
           </geometry>
-          <origin xyz="0.0 0.0 0.0" rpy="${PI / 2} 0.0 0.0" />
+          <origin xyz="0 0 0" rpy="${PI/2} 0 0" />
         </collision>
-        <xacro:cylinder_inertial_matrix m="${wheel_m}" r="${wheel_radius}" h="${wheel_length}" />
+        <xacro:cylinder_inertial_matrix m="${wheel_m}" r="${wheel_radius}" h="${wheel_length}"/>
       </link>
-      <joint name="${name}_wheel2base_link" type="continuous">
-        <parent link="base_link" />
-        <child link="${name}_wheel" />
-        <origin xyz="0 ${flag * base_link_radius} ${-(earth_space + base_link_length / 2 - wheel_radius) }" />
-        <axis xyz="0 1 0" />
+      <joint name="${name}_wheel_joint" type="continuous">
+        <parent link="base_link"/>
+        <child link="${name}_wheel"/>
+        <origin xyz="${x} ${y} ${-(earth_space + base_link_length/2 - wheel_radius)}" rpy="0 0 0"/>
+        <axis xyz="0 1 0"/>
       </joint>
       <gazebo reference="${name}_wheel">
-        <material>Gazebo/Red</material>
+        <material>Gazebo/yellow</material>
       </gazebo>
     </xacro:macro>
-    <xacro:add_wheels name="left" flag="1" />
-    <xacro:add_wheels name="right" flag="-1" />
-    <!-- 支撑轮 -->
-    <!-- 支撑轮属性 -->
-    <xacro:property name="support_wheel_radius" value="0.0075" /> <!-- 支撑轮半径 -->
-    <xacro:property name="support_wheel_m" value="0.03" /> <!-- 质量  -->
-    <!-- 支撑轮宏 -->
-    <xacro:macro name="add_support_wheel" params="name flag" >
-      <link name="${name}_wheel">
-        <visual>
-            <geometry>
-                <sphere radius="${support_wheel_radius}" />
-            </geometry>
-            <origin xyz="0 0 0" rpy="0 0 0" />
-            <material name="black" />
-        </visual>
-        <collision>
-            <geometry>
-                <sphere radius="${support_wheel_radius}" />
-            </geometry>
-            <origin xyz="0 0 0" rpy="0 0 0" />
-        </collision>
-        <xacro:sphere_inertial_matrix m="${support_wheel_m}" r="${support_wheel_radius}" />
-      </link>
-      <joint name="${name}_wheel2base_link" type="continuous">
-          <parent link="base_link" />
-          <child link="${name}_wheel" />
-          <origin xyz="${flag * (base_link_radius - support_wheel_radius)} 0 ${-(base_link_length / 2 + earth_space / 2)}" />
-          <axis xyz="1 1 1" />
-      </joint>
-      <gazebo reference="${name}_wheel">
-        <material>Gazebo/Red</material>
-      </gazebo>
-    </xacro:macro>
-    <xacro:add_support_wheel name="front" flag="1" />
-    <xacro:add_support_wheel name="back" flag="-1" />
+    <!-- 四个角生成麦轮 -->
+    <xacro:add_wheel name="front_left"  x="${ wheel_x_offset}"  y="${ wheel_y_offset}"/>
+    <xacro:add_wheel name="front_right" x="${ wheel_x_offset}"  y="-${ wheel_y_offset}"/>
+    <xacro:add_wheel name="rear_left"   x="-${wheel_x_offset}" y="${ wheel_y_offset}"/>
+    <xacro:add_wheel name="rear_right"  x="-${wheel_x_offset}" y="-${wheel_y_offset}"/>
+  </xacro:macro>
 </robot>

File: robot_gazebo/urdf/robot.urdf (robot description, URDF)
Before this commit: robot my_robot, 9 links, 8 joints
Links:
- removed link back_wheel
- removed link base_footprint
- removed link front_wheel
- removed link left_wheel
- removed link right_wheel
- added link front_left_wheel, mass 0.1; collision cylinder length=0.02 radius=0.0325; visual cylinder length=0.02 radius=0.0325
- added link front_right_wheel, mass 0.1; collision cylinder length=0.02 radius=0.0325; visual cylinder length=0.02 radius=0.0325
- added link rear_left_wheel, mass 0.1; collision cylinder length=0.02 radius=0.0325; visual cylinder length=0.02 radius=0.0325
- added link rear_right_wheel, mass 0.1; collision cylinder length=0.02 radius=0.0325; visual cylinder length=0.02 radius=0.0325
- link base_link: mass 0.5 -> None; geometry visual cylinder length=0.08 radius=0.1
- link support: geometry collision cylinder length=0.05 radius=0.01; visual cylinder length=0.05 radius=0.01
Joints:
- removed joint back_wheel2base_link
- removed joint base_link2base_footprint
- removed joint front_wheel2base_link
- removed joint left_wheel2base_link
- removed joint right_wheel2base_link
- added joint front_left_wheel_joint: type continuous, parent base_link, child front_left_wheel, origin xyz=0.12 0.1 -0.0225 rpy=0 0 0, axis 0 1 0
- added joint front_right_wheel_joint: type continuous, parent base_link, child front_right_wheel, origin xyz=0.12 -0.1 -0.0225 rpy=0 0 0, axis 0 1 0
- added joint rear_left_wheel_joint: type continuous, parent base_link, child rear_left_wheel, origin xyz=-0.12 0.1 -0.0225 rpy=0 0 0, axis 0 1 0
- added joint rear_right_wheel_joint: type continuous, parent base_link, child rear_right_wheel, origin xyz=-0.12 -0.1 -0.0225 rpy=0 0 0, axis 0 1 0
- joint laser2support: origin xyz=0.0 0.0 0.1 -> xyz=0.0 0.0 0.05
- joint support2base_link: origin xyz=0.0 0.0 0.11499999999999999 -> xyz=0.0 0.0 0.065

File: robot_gazebo/urdf/robot.urdf.xacro (robot description, xacro)
@@ -1,8 +1,20 @@
 <robot name="my_robot" xmlns:xacro="http://wiki.ros.org/xacro">
+    <!-- 全局参数 -->
+    <xacro:property name="PI" value="3.1415926"/>
+    <xacro:property name="base_link_length" value="0.08"/>
+    <xacro:property name="base_link_radius" value="0.1"/>
+    <xacro:property name="wheel_radius" value="0.0325"/>
+    <xacro:property name="wheel_length" value="0.02"/>
+    <xacro:property name="wheel_x_offset" value="0.12"/>
+    <xacro:property name="wheel_y_offset" value="0.10"/>
+    <xacro:property name="earth_space" value="0.015"/>
+    <xacro:property name="base_link_m" value="0.5"/>
+    <xacro:property name="wheel_m" value="0.1"/>
+    <xacro:property name="camera_height" value="0.05"/>
+    <!-- 引入 xacro 文件 -->
     <xacro:include filename="cylinder_inertial_matrix.urdf.xacro" />
-    <!-- <xacro:include filename="my_head.urdf.xacro" /> -->
     <xacro:include filename="my_base.urdf.xacro" />
+    <xacro:include filename="move.urdf.xacro" />
     <xacro:include filename="my_camera.urdf.xacro" />
     <xacro:include filename="my_laser.urdf.xacro" />
-    <xacro:include filename="move.urdf.xacro" />
 </robot>
