Commit message: update robot in gazebo without ROSlink

File: robot_gazebo/urdf/robot.urdf (robot description, URDF)
Before this commit: robot mycar, 1 links, 0 joints
Links:
- added link back_wheel, mass 0.03; collision sphere radius=0.0075; visual sphere radius=0.0075
- added link base_footprint; visual sphere radius=0.001
- added link camera, mass 0.01; collision box size=0.01 0.025 0.025; visual box size=0.01 0.025 0.025
- added link front_wheel, mass 0.03; collision sphere radius=0.0075; visual sphere radius=0.0075
- added link laser, mass 0.1; collision cylinder length=0.05 radius=0.03; visual cylinder length=0.05 radius=0.03
- added link left_wheel, mass 0.05; collision cylinder length=0.015 radius=0.0325; visual cylinder length=0.015 radius=0.0325
- added link right_wheel, mass 0.05; collision cylinder length=0.015 radius=0.0325; visual cylinder length=0.015 radius=0.0325
- added link support, mass 0.02; collision cylinder length=0.15 radius=0.01; visual cylinder length=0.15 radius=0.01
- link base_link: mass 6 -> 0.5; geometry collision cylinder length=0.08 radius=0.1; visual cylinder length=0.08 radius=0.1
Joints:
- added joint back_wheel2base_link: type continuous, parent base_link, child back_wheel, origin xyz=-0.0925 0 -0.0475, axis 1 1 1
- added joint base_link2base_footprint: type fixed, parent base_footprint, child base_link, origin xyz=0 0 0.055
- added joint camera2base_link: type fixed, parent base_link, child camera, origin xyz=0.08 0.0 0.052500000000000005
- added joint front_wheel2base_link: type continuous, parent base_link, child front_wheel, origin xyz=0.0925 0 -0.0475, axis 1 1 1
- added joint laser2support: type fixed, parent support, child laser, origin xyz=0.0 0.0 0.1
- added joint left_wheel2base_link: type continuous, parent base_link, child left_wheel, origin xyz=0 0.1 -0.0225, axis 0 1 0
- added joint right_wheel2base_link: type continuous, parent base_link, child right_wheel, origin xyz=0 -0.1 -0.0225, axis 0 1 0
- added joint support2base_link: type fixed, parent base_link, child support, origin xyz=0.0 0.0 0.11499999999999999

Commit message: complete monitor

File: robot_gazebo/urdf/robot.urdf (robot description, URDF)
Before this commit: robot my_robot, 8 links, 7 joints
Links:
- link front_left_wheel: mass 0.1 -> 0.05; geometry collision cylinder length=0.02 radius=0.05; visual cylinder length=0.02 radius=0.05
- link front_right_wheel: mass 0.1 -> 0.05; geometry collision cylinder length=0.02 radius=0.05; visual cylinder length=0.02 radius=0.05
- link rear_left_wheel: mass 0.1 -> 0.05; geometry collision cylinder length=0.02 radius=0.05; visual cylinder length=0.02 radius=0.05
- link rear_right_wheel: mass 0.1 -> 0.05; geometry collision cylinder length=0.02 radius=0.05; visual cylinder length=0.02 radius=0.05
Joints:
- joint front_left_wheel_joint: origin xyz=0.12 0.1 -0.0225 rpy=0 0 0 -> xyz=0.05 0.05 -0.0049999999999999975 rpy=0 0 0
- joint front_right_wheel_joint: origin xyz=0.12 -0.1 -0.0225 rpy=0 0 0 -> xyz=0.05 -0.05 -0.0049999999999999975 rpy=0 0 0
- joint rear_left_wheel_joint: origin xyz=-0.12 0.1 -0.0225 rpy=0 0 0 -> xyz=-0.05 0.05 -0.0049999999999999975 rpy=0 0 0
- joint rear_right_wheel_joint: origin xyz=-0.12 -0.1 -0.0225 rpy=0 0 0 -> xyz=-0.05 -0.05 -0.0049999999999999975 rpy=0 0 0

File: robot_gazebo/urdf/robot.urdf.xacro (robot description, xacro)
@@ -4,11 +4,11 @@
     <xacro:property name="base_link_length" value="0.08"/>
     <xacro:property name="base_link_radius" value="0.1"/>
-    <xacro:property name="wheel_radius" value="0.0325"/>
+    <xacro:property name="wheel_radius" value="0.04"/>
     <xacro:property name="wheel_length" value="0.02"/>
-    <xacro:property name="wheel_x_offset" value="0.12"/>
-    <xacro:property name="wheel_y_offset" value="0.10"/>
+    <xacro:property name="wheel_x_offset" value="0.05"/>
+    <xacro:property name="wheel_y_offset" value="0.05"/>
     <xacro:property name="earth_space" value="0.015"/>
-    <xacro:property name="base_link_m" value="0.5"/>
-    <xacro:property name="wheel_m" value="0.1"/>
+    <xacro:property name="base_link_m" value="0.2"/>
+    <xacro:property name="wheel_m" value="0.05"/>
     <xacro:property name="camera_height" value="0.05"/>
     <!-- 引入 xacro 文件 -->
@@ -18,3 +18,10 @@
     <xacro:include filename="my_camera.urdf.xacro" />
     <xacro:include filename="my_laser.urdf.xacro" />
+    <!-- 加载绝对位姿获取插件 -->
+    <gazebo>
+      <plugin name="odom_plugin" filename="libodom_plugin.so">
+        <topic_name>/absolute_pose</topic_name>
+        <publish_rate>50</publish_rate>
+      </plugin>
+    </gazebo>
 </robot>
