Commit message: fix tf in bsp

File: robot_gazebo/urdf/my_base.urdf.xacro (robot description, xacro)
@@ -35,4 +35,13 @@
           </geometry>
           <origin xyz="0 0 0" rpy="${PI/2} 0 0" />
+          <!-- 添加摩擦力 -->
+          <surface>
+            <friction>
+              <ode>
+                <mu>0.2</mu>      <!-- 主摩擦系数 -->
+                <mu2>0.2</mu2>    <!-- 次摩擦系数 -->
+              </ode>
+            </friction>
+          </surface>
         </collision>
         <xacro:cylinder_inertial_matrix m="${wheel_m}" r="${wheel_radius}" h="${wheel_length}"/>

File: robot_gazebo/urdf/robot.urdf (robot description, URDF)
Before this commit: robot my_robot, 8 links, 7 joints
Links:
- link front_left_wheel: mass 0.05 -> 0.1; geometry collision cylinder length=0.02 radius=0.04; visual cylinder length=0.02 radius=0.04
- link front_right_wheel: mass 0.05 -> 0.1; geometry collision cylinder length=0.02 radius=0.04; visual cylinder length=0.02 radius=0.04
- link rear_left_wheel: mass 0.05 -> 0.1; geometry collision cylinder length=0.02 radius=0.04; visual cylinder length=0.02 radius=0.04
- link rear_right_wheel: mass 0.05 -> 0.1; geometry collision cylinder length=0.02 radius=0.04; visual cylinder length=0.02 radius=0.04
Joints:
- joint front_left_wheel_joint: origin xyz=0.05 0.05 -0.0049999999999999975 rpy=0 0 0 -> xyz=0.1 0.1 -0.010000000000000002 rpy=0 0 0
- joint front_right_wheel_joint: origin xyz=0.05 -0.05 -0.0049999999999999975 rpy=0 0 0 -> xyz=0.1 -0.1 -0.010000000000000002 rpy=0 0 0
- joint rear_left_wheel_joint: origin xyz=-0.05 0.05 -0.0049999999999999975 rpy=0 0 0 -> xyz=-0.1 0.1 -0.010000000000000002 rpy=0 0 0
- joint rear_right_wheel_joint: origin xyz=-0.05 -0.05 -0.0049999999999999975 rpy=0 0 0 -> xyz=-0.1 -0.1 -0.010000000000000002 rpy=0 0 0

File: robot_gazebo/urdf/robot.urdf.xacro (robot description, xacro)
@@ -6,9 +6,9 @@
     <xacro:property name="wheel_radius" value="0.04"/>
     <xacro:property name="wheel_length" value="0.02"/>
-    <xacro:property name="wheel_x_offset" value="0.05"/>
-    <xacro:property name="wheel_y_offset" value="0.05"/>
-    <xacro:property name="earth_space" value="0.015"/>
+    <xacro:property name="wheel_x_offset" value="0.1"/>
+    <xacro:property name="wheel_y_offset" value="0.1"/>
+    <xacro:property name="earth_space" value="0.010"/>
     <xacro:property name="base_link_m" value="0.2"/>
-    <xacro:property name="wheel_m" value="0.05"/>
+    <xacro:property name="wheel_m" value="0.1"/>
     <xacro:property name="camera_height" value="0.05"/>
     <!-- 引入 xacro 文件 -->

Commit message: update

File: robot_gazebo/urdf/my_base.urdf.xacro (robot description, xacro)
@@ -8,6 +8,15 @@
         <color rgba="1.0 1.0 0.0 1.0" />
     </material>
+    <!-- 虚拟的 root link（无质量，无惯性） -->
+    <link name="base_footprint"/>
+    <!-- 原 base_link 是 base_footprint 的子链接 -->
+    <joint name="base_footprint_to_base_link" type="fixed">
+      <parent link="base_footprint"/>
+      <child link="base_link"/>
+      <origin xyz="0 0 ${wheel_radius + earth_space}" rpy="0 0 0"/>
+    </joint>
     <!-- 底盘主体 -->
     <link name="base_link">
+      <!-- 可视化 -->
       <visual>
         <geometry>
@@ -19,4 +28,23 @@
         </material>
       </visual>
+      <!-- 碰撞体 -->
+      <collision>
+        <geometry>
+          <cylinder radius="${base_link_radius}" length="${base_link_length}" />
+        </geometry>
+        <origin xyz="0 0 0" rpy="0 0 0" />
+      </collision>
+      <!-- 惯性矩阵 -->
+      <inertial>
+        <mass value="${base_link_m}"/>
+        <origin xyz="0 0 0" rpy="0 0 0"/>
+        <inertia
+          ixx="${(base_link_m * (3 * base_link_radius * base_link_radius + base_link_length * base_link_length)) / 12.0}"
+          ixy="0"
+          ixz="0"
+          iyy="${(base_link_m * (3 * base_link_radius * base_link_radius + base_link_length * base_link_length)) / 12.0}"
+          iyz="0"
+          izz="${(base_link_m * base_link_radius * base_link_radius) / 2.0}"/>
+      </inertial>
     </link>
     <!-- 四个驱动轮宏 -->

File: robot_gazebo/urdf/robot.urdf (robot description, URDF)
Before this commit: robot my_robot, 8 links, 7 joints
Links:
- added link base_footprint
- link base_link: mass None -> 0.2; geometry collision cylinder length=0.08 radius=0.1; visual cylinder length=0.08 radius=0.1
Joints:
- added joint base_footprint_to_base_link: type fixed, parent base_footprint, child base_link, origin xyz=0 0 0.05 rpy=0 0 0

File: robot_gazebo/urdf/robot.urdf.xacro (robot description, xacro)
@@ -4,8 +4,8 @@
     <xacro:property name="base_link_length" value="0.08"/>
     <xacro:property name="base_link_radius" value="0.1"/>
-    <xacro:property name="wheel_radius" value="0.04"/>
+    <xacro:property name="wheel_radius" value="0.0325"/>
     <xacro:property name="wheel_length" value="0.02"/>
-    <xacro:property name="wheel_x_offset" value="0.1"/>
-    <xacro:property name="wheel_y_offset" value="0.1"/>
+    <xacro:property name="wheel_x_offset" value="0.08"/>
+    <xacro:property name="wheel_y_offset" value="0.08"/>
     <xacro:property name="earth_space" value="0.010"/>
     <xacro:property name="base_link_m" value="0.2"/>

Commit message: fix all bugs in gazebo

File: robot_gazebo/urdf/my_base.urdf.xacro (robot description, xacro)
@@ -45,5 +45,5 @@
           iyy="${(base_link_m * (3 * base_link_radius * base_link_radius + base_link_length * base_link_length)) / 12.0}"
           iyz="0"
-          izz="${(base_link_m * base_link_radius * base_link_radius) / 2.0}"/>
+          izz="0.1"/>
       </inertial>
     </link>

File: robot_gazebo/urdf/robot.urdf (robot description, URDF)
Before this commit: robot my_robot, 9 links, 8 joints
Links:
- link base_link: mass 0.2 -> 2.0
- link front_left_wheel: geometry collision cylinder length=0.02 radius=0.0325; visual cylinder length=0.02 radius=0.0325
- link front_right_wheel: geometry collision cylinder length=0.02 radius=0.0325; visual cylinder length=0.02 radius=0.0325
- link rear_left_wheel: geometry collision cylinder length=0.02 radius=0.0325; visual cylinder length=0.02 radius=0.0325
- link rear_right_wheel: geometry collision cylinder length=0.02 radius=0.0325; visual cylinder length=0.02 radius=0.0325
Joints:
- joint base_footprint_to_base_link: origin xyz=0 0 0.05 rpy=0 0 0 -> xyz=0 0 0.0425 rpy=0 0 0
- joint front_left_wheel_joint: origin xyz=0.1 0.1 -0.010000000000000002 rpy=0 0 0 -> xyz=0.08 0.08 -0.0175 rpy=0 0 0
- joint front_right_wheel_joint: origin xyz=0.1 -0.1 -0.010000000000000002 rpy=0 0 0 -> xyz=0.08 -0.08 -0.0175 rpy=0 0 0
- joint rear_left_wheel_joint: origin xyz=-0.1 0.1 -0.010000000000000002 rpy=0 0 0 -> xyz=-0.08 0.08 -0.0175 rpy=0 0 0
- joint rear_right_wheel_joint: origin xyz=-0.1 -0.1 -0.010000000000000002 rpy=0 0 0 -> xyz=-0.08 -0.08 -0.0175 rpy=0 0 0

File: robot_gazebo/urdf/robot.urdf.xacro (robot description, xacro)
@@ -9,5 +9,5 @@
     <xacro:property name="wheel_y_offset" value="0.08"/>
     <xacro:property name="earth_space" value="0.010"/>
-    <xacro:property name="base_link_m" value="0.2"/>
+    <xacro:property name="base_link_m" value="2.0"/>
     <xacro:property name="wheel_m" value="0.1"/>
     <xacro:property name="camera_height" value="0.05"/>
@@ -33,5 +33,5 @@
         <odometryFrame>odom</odometryFrame>
         <odometryRate>50.0</odometryRate>
-        <robotBaseFrame>base_link</robotBaseFrame>
+        <robotBaseFrame>base_footprint</robotBaseFrame>
         <update_rate>50</update_rate>
       </plugin>

Commit message: finish

File: robot_gazebo/urdf/my_base.urdf.xacro (robot description, xacro)
@@ -67,6 +67,6 @@
             <friction>
               <ode>
-                <mu>0.2</mu>      <!-- 主摩擦系数 -->
-                <mu2>0.2</mu2>    <!-- 次摩擦系数 -->
+                <mu>1.0</mu>      <!-- 主摩擦系数 -->
+                <mu2>1.0</mu2>    <!-- 次摩擦系数 -->
               </ode>
             </friction>

File: robot_gazebo/urdf/my_camera.urdf.xacro (robot description, xacro)
@@ -1,3 +1,3 @@
-<!-- 摄像头相关的 xacro 文件 -->
+<!-- 摄像头 -->
 <robot name="my_camera" xmlns:xacro="http://wiki.ros.org/xacro">
     <!-- 属性 -->
@@ -5,32 +5,90 @@
     <xacro:property name="camera_width" value="0.025" /> <!-- 摄像头宽度(y) -->
     <xacro:property name="camera_height" value="0.025" /> <!-- 摄像头高度(z) -->
-    <xacro:property name="camera_x" value="0.08" /> <!-- 摄像头安装的x坐标 -->
-    <xacro:property name="camera_y" value="0.0" /> <!-- 摄像头安装的y坐标 -->
-    <xacro:property name="camera_z" value="${base_link_length / 2 + camera_height / 2}" /> <!-- 摄像头安装的z坐标:底盘高度 / 2 + 摄像头高度 / 2  -->
     <xacro:property name="camera_m" value="0.01" /> <!-- 摄像头质量 -->
-    <!-- 摄像头关节以及link -->
-    <link name="camera">
-        <visual>
-            <geometry>
-                <box size="${camera_length} ${camera_width} ${camera_height}" />
-            </geometry>
-            <origin xyz="0.0 0.0 0.0" rpy="0.0 0.0 0.0" />
-            <material name="black" />
-        </visual>
-        <collision>
-            <geometry>
-                <box size="${camera_length} ${camera_width} ${camera_height}" />
-            </geometry>
-            <origin xyz="0.0 0.0 0.0" rpy="0.0 0.0 0.0" />
-        </collision>
-        <xacro:Box_inertial_matrix m="${camera_m}" l="${camera_length}" w="${camera_width}" h="${camera_height}" />
-    </link>
-    <joint name="camera2base_link" type="fixed">
-        <parent link="base_link" />
-        <child link="camera" />
-        <origin xyz="${camera_x} ${camera_y} ${camera_z}" />
-    </joint>
-    <gazebo reference="camera">
-        <material>Gazebo/Blue</material>
-    </gazebo>
+    <!-- 安装位置 -->
+    <xacro:property name="camera_x" value="0.0" />  <!-- 与车体中心对齐 -->
+    <xacro:property name="camera_y_offset" value="0.08" />  <!-- 两侧偏移距离 -->
+    <xacro:property name="camera_z" value="${base_link_length / 2 + camera_height / 2}" />
+    <!-- 摄像头宏定义 - 可重复使用 -->
+    <xacro:macro name="camera_module" params="name parent_link x y z yaw">
+        <!-- 摄像头 Link -->
+        <link name="${name}">
+            <visual>
+                <geometry>
+                    <box size="${camera_length} ${camera_width} ${camera_height}" />
+                </geometry>
+                <origin xyz="0 0 0" rpy="0 0 0" />
+                <material name="camera_blue">
+                    <color rgba="0.2 0.5 0.8 1.0" />
+                </material>
+            </visual>
+            <collision>
+                <geometry>
+                    <box size="${camera_length} ${camera_width} ${camera_height}" />
+                </geometry>
+                <origin xyz="0 0 0" rpy="0 0 0" />
+            </collision>
+            <xacro:Box_inertial_matrix m="${camera_m}" l="${camera_length}" w="${camera_width}" h="${camera_height}" />
+        </link>
+        <!-- 摄像头 Joint -->
+        <joint name="${name}_joint" type="fixed">
+            <parent link="${parent_link}" />
+            <child link="${name}" />
+            <origin xyz="${x} ${y} ${z}" rpy="0 0 ${yaw}" />
+        </joint>
+        <!-- Gazebo 材质 -->
+        <gazebo reference="${name}">
+            <material>Gazebo/Blue</material>
+        </gazebo>
+        <!-- Gazebo 摄像头传感器插件 -->
+        <gazebo reference="${name}">
+            <sensor type="camera" name="${name}_sensor">
+                <update_rate>30.0</update_rate>
+                <visualize>true</visualize>  <!-- 在 Gazebo 中显示摄像头视锥 -->
+                <camera name="${name}">
+                    <horizontal_fov>1.6</horizontal_fov>  <!-- 90度视角 = 1.6 弧度 -->
+                    <image>
+                        <width>1280</width>  <!-- 720p 宽度 -->
+                        <height>720</height>  <!-- 720p 高度 -->
+                        <format>R8G8B8</format>
+                    </image>
+                    <clip>
+                        <near>0.02</near>
+                        <far>10.0</far>
+                    </clip>
+                    <noise>
+                        <type>gaussian</type>
+                        <mean>0.0</mean>
+                        <stddev>0.007</stddev>
+                    </noise>
+                </camera>
+                <plugin name="${name}_controller" filename="libgazebo_ros_camera.so">
+                    <ros>
+                        <namespace></namespace>
+                        <remapping>image_raw:=${name}/image_raw</remapping>
+                        <remapping>camera_info:=${name}/camera_info</remapping>
+                    </ros>
+                    <camera_name>${name}</camera_name>
+                    <frame_name>${name}</frame_name>
+                    <hack_baseline>0.07</hack_baseline>
+                </plugin>
+            </sensor>
+        </gazebo>
+    </xacro:macro>
+    <!-- 左侧摄像头 - 朝左 (yaw = 1.5708 = 90度) -->
+    <xacro:camera_module
+        name="camera1"
+        parent_link="base_link"
+        x="${camera_x}"
+        y="${camera_y_offset}"
+        z="${camera_z}"
+        yaw="1.5708" />
+    <!-- 右侧摄像头 - 朝右 (yaw = -1.5708 = -90度) -->
+    <xacro:camera_module
+        name="camera2"
+        parent_link="base_link"
+        x="${camera_x}"
+        y="${-camera_y_offset}"
+        z="${camera_z}"
+        yaw="-1.5708" />
 </robot>

File: robot_gazebo/urdf/my_laser.urdf.xacro (robot description, xacro)
@@ -65,3 +65,32 @@
         <material>Gazebo/Black</material>
     </gazebo>
+    <!-- 雷达传感器仿真插件 -->
+    <gazebo reference="laser">
+        <sensor name="laser_sensor" type="ray">
+            <visualize>false</visualize>
+            <update_rate>10</update_rate>
+            <ray>
+                <scan>
+                    <horizontal>
+                        <samples>720</samples>
+                        <resolution>1</resolution>
+                        <min_angle>-3.14159</min_angle>
+                        <max_angle>3.14159</max_angle>
+                    </horizontal>
+                </scan>
+                <range>
+                    <min>0.15</min>
+                    <max>12.0</max>
+                    <resolution>0.01</resolution>
+                </range>
+            </ray>
+            <plugin name="gazebo_ros_laser" filename="libgazebo_ros_ray_sensor.so">
+                <ros>
+                    <remapping>~/out:=scan</remapping>
+                </ros>
+                <output_type>sensor_msgs/LaserScan</output_type>
+                <frame_name>laser</frame_name>
+            </plugin>
+        </sensor>
+    </gazebo>
 </robot>

File: robot_gazebo/urdf/robot.urdf (robot description, URDF)
Before this commit: robot my_robot, 9 links, 8 joints
Links:
- removed link camera
- added link camera1, mass 0.01; collision box size=0.01 0.025 0.025; visual box size=0.01 0.025 0.025
- added link camera2, mass 0.01; collision box size=0.01 0.025 0.025; visual box size=0.01 0.025 0.025
Joints:
- removed joint camera2base_link
- added joint camera1_joint: type fixed, parent base_link, child camera1, origin xyz=0.0 0.08 0.052500000000000005 rpy=0 0 1.5708
- added joint camera2_joint: type fixed, parent base_link, child camera2, origin xyz=0.0 -0.08 0.052500000000000005 rpy=0 0 -1.5708

File: robot_gazebo/urdf/robot.urdf.xacro (robot description, xacro)
@@ -37,35 +37,3 @@
       </plugin>
     </gazebo>
-    <!-- 雷达传感器仿真插件 -->
-  <gazebo reference="laser">
-      <sensor type="ray" name="rplidar">
-          <pose>0 0 0 0 0 0</pose>
-          <visualize>false</visualize> <!-- Gazebo中显示雷达探测线 -->
-          <update_rate>10</update_rate>
-          <ray>
-              <scan>
-                  <horizontal>
-                      <samples>360</samples>
-                      <resolution>1</resolution>
-                      <min_angle>-3.14159</min_angle>
-                      <max_angle>3.14159</max_angle>
-                  </horizontal>
-              </scan>
-              <range>
-                  <min>0.15</min>
-                  <max>12.0</max>
-                  <resolution>0.01</resolution>
-              </range>
-              <noise>
-                  <type>gaussian</type>
-                  <mean>0.0</mean>
-                  <stddev>0.01</stddev>
-              </noise>
-          </ray>
-          <plugin name="gazebo_ros_rplidar_controller" filename="libgazebo_ros_laser.so">
-              <topicName>/scan</topicName>
-              <frameName>laser</frameName>
-          </plugin>
-      </sensor>
-  </gazebo>
 </robot>
